Commit message: feat: 在rviz2中实现了相机模型的注入

File: franka_description/robots/sim/dual_panda_arm_sim.urdf.xacro (robot description, xacro)
@@ -36,4 +36,48 @@
     <xacro:hand ns="$(arg arm_id_2)" rpy="0 0 ${-pi/4}" connected_to="$(arg arm_id_2)_link8" safety_distance="0.03"/>
   </xacro:if>
+  <!-- left_arm_cam -->
+  <joint name="$(arg arm_id_1)_camera_joint" type="fixed">
+    <parent link="$(arg arm_id_1)_hand"/>
+    <child link="left_real_camera"/>
+    <origin xyz="0 0 0" rpy="0 0 0"/>
+  </joint>
+  <link name="left_real_camera">
+    <visual>
+      <origin xyz="0 0 0" rpy="0 0 0"/>
+      <geometry>
+        <mesh filename="package://franka_description/meshes/visual/camera_part1.stl" scale="0.001 0.001 0.001"/>
+      </geometry>
+      <material name="cam_L1"><color rgba="1.0 1.0 1.0 1.0"/></material>
+    </visual>
+    <visual>
+      <origin xyz="0 0 0" rpy="0 0 0"/>
+      <geometry>
+        <mesh filename="package://franka_description/meshes/visual/camera_part2.stl" scale="0.001 0.001 0.001"/>
+      </geometry>
+      <material name="cam_L2"><color rgba="1.0 1.0 1.0 1.0"/></material>
+    </visual>
+  </link>
+  <!-- right_arm_cam -->
+  <joint name="$(arg arm_id_2)_camera_joint" type="fixed">
+    <parent link="$(arg arm_id_2)_hand"/>
+    <child link="right_real_camera"/>
+    <origin xyz="0 0 0" rpy="0 0 0"/>
+  </joint>
+  <link name="right_real_camera">
+    <visual>
+      <origin xyz="0 0 0" rpy="0 0 0"/>
+      <geometry>
+        <mesh filename="package://franka_description/meshes/visual/camera_part1.stl" scale="0.001 0.001 0.001"/>
+      </geometry>
+      <material name="cam_R1"><color rgba="1.0 1.0 1.0 1.0"/></material>
+    </visual>
+    <visual>
+      <origin xyz="0 0 0" rpy="0 0 0"/>
+      <geometry>
+        <mesh filename="package://franka_description/meshes/visual/camera_part2.stl" scale="0.001 0.001 0.001"/>
+      </geometry>
+      <material name="cam_R2"><color rgba="1.0 1.0 1.0 1.0"/></material>
+    </visual>
+  </link>
   <xacro:include filename="$(find franka_description)/robots/sim/dual_panda_arm_sim.ros2_control.xacro"/>
   <xacro:dual_panda_mjros_ros2_control

Commit message: feat: 为左右相机添加碰撞体积以增强物理仿真

File: franka_description/robots/sim/dual_panda_arm_sim.urdf.xacro (robot description, xacro)
@@ -57,4 +57,16 @@
       <material name="cam_L2"><color rgba="1.0 1.0 1.0 1.0"/></material>
     </visual>
+    <collision>
+      <origin xyz="0.110674 0 0.043860" rpy="0 0 0"/>
+      <geometry>
+        <sphere radius="0.034"/>
+      </geometry>
+    </collision>
+    <collision>
+      <origin xyz="0.072659 0.000255 0.001474" rpy="0 0 0"/>
+      <geometry>
+        <sphere radius="0.032"/>
+      </geometry>
+    </collision>
   </link>
   <!-- right_arm_cam -->
@@ -79,4 +91,16 @@
       <material name="cam_R2"><color rgba="1.0 1.0 1.0 1.0"/></material>
     </visual>
+    <collision>
+      <origin xyz="0.110674 0.0 0.043860" rpy="0 0 0"/>
+      <geometry>
+        <sphere radius="0.034"/>
+      </geometry>
+    </collision>
+    <collision>
+      <origin xyz="0.072659 0.000255 0.001474" rpy="0 0 0"/>
+      <geometry>
+        <sphere radius="0.032"/>
+      </geometry>
+    </collision>
   </link>
   <xacro:include filename="$(find franka_description)/robots/sim/dual_panda_arm_sim.ros2_control.xacro"/>

Commit message: fix: 修正左右相机碰撞体积的坐标值以提高物理仿真精度

File: franka_description/robots/sim/dual_panda_arm_sim.urdf.xacro (robot description, xacro)
@@ -64,5 +64,5 @@
     </collision>
     <collision>
-      <origin xyz="0.072659 0.000255 0.001474" rpy="0 0 0"/>
+      <origin xyz="0.072659 0 0.001474" rpy="0 0 0"/>
       <geometry>
         <sphere radius="0.032"/>
@@ -98,5 +98,5 @@
     </collision>
     <collision>
-      <origin xyz="0.072659 0.000255 0.001474" rpy="0 0 0"/>
+      <origin xyz="0.072659 0.0 0.001474" rpy="0 0 0"/>
       <geometry>
         <sphere radius="0.032"/>
